File: hardware/Kicad/Pioneer Controller V2/Pioneer Controller V2.kicad_pcb (KiCad board)
At the start: 2 copper layers, 72 x 98.8 mm, 32 parts, among them J1 Sensor Connector, J2 Power (IN), J4 Conn_Coaxial, SW1 SW_Push, SW2 SW_Push, SW5 SW_DIP_x02, U1 ESP32-S3, U2 2821, U3 DS3231_Precision_RTC, U4 RFM95W_LoRa_Radio_Transceiver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

Commit message: updated PCBS
Parts:
- removed D2: LED, LED_SMD:LED_1206_3216Metric
- removed R4: R5k, Resistor_SMD:R_1206_3216Metric
- added U8: MicroSD_Breakout, Adafruit_Sensors:MicroSD_Breakout, B.Cu at (73.2, 117.1)
- moved C7 8.75 mm to (87.2, 92.0)
- moved SW5 1.80 mm to (65.8, 84.7)
- moved U3 0.20 mm to (69.2, 41.0)
Connections:
- net /CS renamed /CS0
- U1 pad D5: /LED2 -> /CS1
- U2 pad 21: /LED2 -> /LED1
- U2 pad 24: /LED1 -> /CS1
Routing:
- net /CS1: track 0.00 -> 107.8 mm, vias 0 -> 3
- net /LED2: track 97.2 -> 0.00 mm, vias 2 -> 0
- net /SCK: track 71.5 -> 103.0 mm, vias 1 -> 2
- net /MOSI: track 84.3 -> 114.4 mm
- net /MISO: track 79.0 -> 108.9 mm, vias 3 -> 4
- net +5V: track 85.7 -> 104.8 mm, vias 0 -> 1
- net /RX: track 116.2 -> 132.6 mm
- net /TX: track 120.3 -> 132.2 mm, vias 0 -> 1
- net /LED1: track 120.2 -> 112.6 mm, vias 5 -> 2
- net +3V3: track 226.2 -> 230.8 mm
- net /SW5: track 48.3 -> 51.1 mm, vias 0 -> 1
- net /SW6: track 44.2 -> 46.4 mm, vias 0 -> 1
- net Net-(D2-Pad1): track 2.14 -> 0.00 mm
- net /SW1: track 127.7 -> 129.2 mm
Other:
- board text added: "BME TEMPERATURE SENSOR"
- board text added: "BUTTON 1"
- board text added: "BUTTON 2"
- board text added: "ESP32-S3"
- board text added: "ESP8266"
- board text added: "HAVE YOU HEARD OF THE HIT GAME AMONG US?"
- board text added: "LoRa MODULE"
- board text added: "MICRO SD"
- board text added: "PAT"
- board text added: "PIONEER Radio Communication Module"
- board text added: "POWER IN"
- board text added: "RTC CLOCK"
- board text added: "SENSOR CONNECTOR"
- board text added: "SMA"
