File: hardware/Kicad/Pioneer Controller V2/Pioneer Controller V2.kicad_sch (KiCad schematic)
At the start: 28 parts, among them J1 Sensor Connector, J2 Power (IN), J4 Conn_Coaxial, SW1 SW_Push, SW2 SW_Push, SW5 SW_DIP_x02, U1 ESP32-S3, U2 2821, U3 DS3231_Precision_RTC, U4 RFM95W_LoRa_Radio_Transceiver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

Commit message: updated PCBS
Parts:
- removed D2: LED, LED_SMD:LED_1206_3216Metric, symbol Device:LED
- removed R4: R5k, Resistor_SMD:R_1206_3216Metric, symbol Device:R
- added U8: MicroSD_Breakout, Adafruit_Sensors:MicroSD_Breakout, symbol Adafruit_Files:MicroSD_Breakout
Connections:
- net +5V: now also U8.5V
- net GND: now also U8.GND
- net LED1: now also U2.21 (GPIO12); no longer U2.24 (GPIO0)
- net MISO: now also U8.DO
- net MOSI: now also U8.DI
- net SCK: now also U8.CLK
- net CS renamed CS0
- net LED2 renamed CS1
- net CS1: now also U2.24 (GPIO0), U8.CS; no longer U2.21 (GPIO12)
- no-connect marks 26 -> 27
Other:
- note added: "Micro SD"
- moved on the sheet: D1, R1
