File: hardware/Kicad/Sensor/Sensor.kicad_pcb (KiCad board)
At the start: 2 copper layers, 58.5 x 64 mm, 19 parts, among them J1 Controller Connector, J2 Conn_01x08, J3 Conn_01x08, J4 Conn_01x06, J5 Conn_01x06, J6 Conn_01x04, U1 2821, U2 4Channel_ADC_Breakout, U3 4Channel_ADC_Breakout, U4 4Channel_ADC_Breakout

Commit message: updated PCBS
Parts:
- C1: moved to B.Cu
- U2, U3: moved to F.Cu
- U4: value 4Channel_ADC_Breakout -> MicroSD_Breakout; footprint Adafruit_Sensors:4Channel ADC Breakout -> Adafruit_Sensors:MicroSD_Breakout; moved to F.Cu
- moved U4 66.2 mm to (87.0, 139.3)
- moved J2 63.9 mm to (36.5, 136.5), turned to 0 degrees
- moved R1 58.6 mm to (34.0, 129.5), turned to 90 degrees
- moved J5 56.4 mm to (89.0, 81.0), turned to 180 degrees
- moved J4 56.4 mm to (70.0, 81.0), turned to 180 degrees
- moved R3 55.0 mm to (38.5, 129.5), turned to 90 degrees
- moved J6 51.5 mm to (70.8, 130.0), turned to 180 degrees
- moved J3 48.0 mm to (61.5, 136.5), turned to 0 degrees
- moved R4 44.6 mm to (51.5, 128.0)
- moved R2 41.2 mm to (55.0, 131.0)
- moved U2 39.2 mm to (87.0, 84.2), turned to 0 degrees
- moved U3 36.8 mm to (59.0, 102.0), turned to 180 degrees
- moved U1 28.0 mm to (48.0, 114.0)
- moved J1 26.9 mm to (24.0, 128.2)
- moved C1 22.7 mm to (27.5, 134.5), turned to 90 degrees
Connections:
- J4 pad 1: /A2N -> GND
- J4 pad 2: /A2P -> /A1N
- J4 pad 3: /A1N -> GND
- J5 pad 1: /A4N -> GND
- J5 pad 2: /A4P -> /A2N
- J5 pad 3: /A3N -> GND
- J5 pad 4: /A3P -> /A2P
- J6 pad 1: /A5N -> /A3P
- J6 pad 2: /A5P -> /A3N
- U1 pad 20: unconnected-(U1-Pad20) -> /CS1
- U3 pad A0: /A4N -> unconnected-(U3-PadA0)
- U3 pad A1: /A4P -> unconnected-(U3-PadA1)
Routing:
- net /MISO: track 0.00 -> 57.3 mm
- net /MOSI: track 0.00 -> 56.0 mm, vias 0 -> 1
- net /SCK: track 0.00 -> 51.4 mm, vias 0 -> 1
- net /CS1: track 0.00 -> 44.2 mm
- net /SCL: track 92.8 -> 57.7 mm, vias 2 -> 1
- net /A3P: track 15.0 -> 43.7 mm, vias 0 -> 1
- net /A4N: track 28.5 -> 0.00 mm
- net /SDA: track 85.2 -> 58.5 mm, vias 0 -> 2
- net /A3N: track 18.8 -> 45.3 mm, vias 0 -> 1
- net /A4P: track 22.9 -> 0.00 mm
- net /A2N: track 28.7 -> 7.53 mm
- net +3V3: track 61.0 -> 43.3 mm
- net /A5P: track 17.7 -> 0.00 mm
- net /A5N: track 16.1 -> 0.00 mm
- net /A2P: track 24.6 -> 10.2 mm
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Other:
- board size 58.5 x 64 mm -> 81 x 64 mm

Commit message: updated PCB labels
Other:
- board text added: "ADC MODULE"
- board text added: "ESP8266"
- board text added: "GND"
- board text added: "HAVE YOU HEARD OF THE HIT GAME AMONG US?"
- board text added: "MAIN"
- board text added: "MICRO SD"
- board text added: "PIONEER Sensor Module"
- board text added: "RICK"
Changed lines of the file:
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@@
     (property "Sheetname" "")
     (attr smd)
-    (fp_text reference "J3" (at 8.5 0.25) (layer "F.SilkS")
+    (fp_text reference "J3" (at 8.5 -2.5) (layer "F.SilkS")
       (effects (font (size 1 1) (thickness 0.15)))
     )
@@
       (effects (font (size 1 1) (thickness 0.15)))
     )
-    (fp_text user "${REFERENCE}" (at 8.5 0.25) (layer "F.Fab")
+    (fp_text user "${REFERENCE}" (at 8.5 -2.5) (layer "F.Fab")
       (effects (font (size 1 1) (thickness 0.15)))
     )
@@
     (property "Sheetname" "")
     (attr through_hole)
-    (fp_text reference "U4" (at 0 4.07 180 unlocked) (layer "F.SilkS")
-      (effects (font (size 1 1) (thickness 0.15)))
-    )
-    (fp_text value "MicroSD_Breakout" (at 0 2.5 180 unlocked) (layer "F.Fab")
-      (effects (font (size 1 1) (thickness 0.15)))
-    )
-    (fp_text user "${REFERENCE}" (at 0 4 180 unlocked) (layer "F.Fab")
+    (fp_text reference "U4" (at 11 6.35 180 unlocked) (layer "F.SilkS")
+      (effects (font (size 1 1) (thickness 0.15)))
+    )
+    (fp_text value "MicroSD_Breakout" (at -1 6.32 180 unlocked) (layer "F.Fab")
+      (effects (font (size 1 1) (thickness 0.15)))
+    )
+    (fp_text user "${REFERENCE}" (at 11 6.32 180 unlocked) (layer "F.Fab")
       (effects (font (size 1 1) (thickness 0.15)))
     )
@@
   (gr_line (start 21 136) (end 21 105) (layer "Edge.Cuts") (width 0.1))
   (gr_arc (start 102 136) (mid 100.828427 138.828427) (end 98 140) (layer "Edge.Cuts") (width 0.1))
+  (gr_text "HAVE YOU HEARD OF\nTHE HIT GAME \nAMONG US?" (at 67.5 121.75) (layer "F.SilkS")
+    (effects (font (size 0.5 0.5) (thickness 0.125)))
+  )
+  (gr_text "ADC MODULE" (at 100.5 93 270) (layer "F.SilkS")
+    (effects (font (size 1 1) (thickness 0.15)))
+  )
+  (gr_text "MAIN" (at 26.5 132.5 270) (layer "F.SilkS")
+    (effects (font (size 1 1) (thickness 0.15)))
+  )
+  (gr_text "GND" (at 44.5 138.5 270) (layer "F.SilkS")
+    (effects (font (size 0.8 0.8) (thickness 0.15)))
+  )
+  (gr_text "ADC MODULE" (at 72.5 93 270) (layer "F.SilkS")
+    (effects (font (size 1 1) (thickness 0.15)))
+  )
+  (gr_text "GND" (at 70 76.5 180) (layer "F.SilkS")
+    (effects (font (size 0.8 0.8) (thickness 0.15)))
+  )
+  (gr_text "MICRO SD" (at 90 135 180) (layer "F.SilkS")
+    (effects (font (size 1 1) (thickness 0.15)))
+  )
+  (gr_text "ESP8266" (at 24 114 90) (layer "F.SilkS")
+    (effects (font (size 1 1) (thickness 0.15)))
+  )
+  (gr_text "RICK" (at 86 115) (layer "F.SilkS")
+    (effects (font (size 4 4) (thickness 0.3)))
+  )
+  (gr_text "GND" (at 22 133.5 270) (layer "F.SilkS")
+    (effects (font (size 0.8 0.8) (thickness 0.15)))
+  )
+  (gr_text "GND" (at 69.5 138.5 270) (layer "F.SilkS")
+    (effects (font (size 0.8 0.8) (thickness 0.15)))
+  )
+  (gr_text "GND" (at 89 76.5 180) (layer "F.SilkS")
+    (effects (font (size 0.8 0.8) (thickness 0.15)))
+  )
+  (gr_text "GND" (at 65.5 128) (layer "F.SilkS")
+    (effects (font (size 0.8 0.8) (thickness 0.15)))
+  )
+  (gr_text "PIONEER Sensor Module" (at 89 118) (layer "F.SilkS")
+    (effects (font (size 1 1) (thickness 0.15) italic))
+  )
   (dimension (type aligned) (layer "Dwgs.User")
     (pts (xy 21 134.5) (xy 102 134.5))

Commit message: added extra resistor
Parts:
- added R5: 250R, Resistor_SMD:R_0805_2012Metric, F.Cu at (74.8, 137.1)
Routing:
- net /A3P: track 43.7 -> 54.2 mm
- net /A3N: track 45.3 -> 54.7 mm
Changed lines of the file:
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@@
+    )
+  )
+  (footprint "Resistor_SMD:R_0805_2012Metric" (layer "F.Cu")
+    (at 74.8 137.1 180)
+    (descr "Resistor SMD 0805 (2012 Metric), square (rectangular) end terminal, IPC_7351 nominal, (Body size source: IPC-SM-782 page 72, https://www.pcb-3d.com/wordpress/wp-content/uploads/ipc-sm-782a_amendment_1_and_2.pdf), generated with kicad-footprint-generator")
+    (tags "resistor")
+    (property "Sheetfile" "Sensor.kicad_sch")
+    (property "Sheetname" "")
+    (attr smd)
+    (fp_text reference "R5" (at 0 -1.65) (layer "F.SilkS")
+      (effects (font (size 1 1) (thickness 0.15)))
+    )
+    (fp_text value "250R" (at 0 1.65) (layer "F.Fab")
+      (effects (font (size 1 1) (thickness 0.15)))
+    )
+    (fp_text user "${REFERENCE}" (at 0 0) (layer "F.Fab")
+      (effects (font (size 0.5 0.5) (thickness 0.08)))
+    )
+    (fp_line (start -0.227064 -0.735) (end 0.227064 -0.735) (layer "F.SilkS") (width 0.12))
+    (fp_line (start -0.227064 0.735) (end 0.227064 0.735) (layer "F.SilkS") (width 0.12))
+    (fp_line (start 1.68 -0.95) (end 1.68 0.95) (layer "F.CrtYd") (width 0.05))
+    (fp_line (start -1.68 -0.95) (end 1.68 -0.95) (layer "F.CrtYd") (width 0.05))
+    (fp_line (start 1.68 0.95) (end -1.68 0.95) (layer "F.CrtYd") (width 0.05))
+    (fp_line (start -1.68 0.95) (end -1.68 -0.95) (layer "F.CrtYd") (width 0.05))
+    (fp_line (start 1 -0.625) (end 1 0.625) (layer "F.Fab") (width 0.1))
+    (fp_line (start -1 0.625) (end -1 -0.625) (layer "F.Fab") (width 0.1))
+    (fp_line (start -1 -0.625) (end 1 -0.625) (layer "F.Fab") (width 0.1))
+    (fp_line (start 1 0.625) (end -1 0.625) (layer "F.Fab") (width 0.1))
+    (pad "1" smd roundrect (at -0.9125 0 180) (size 1.025 1.4) (layers "F.Cu" "F.Paste" "F.Mask") (roundrect_rratio 0.243902)
+      (net 22 "/A3P") (pintype "passive"))
+    (pad "2" smd roundrect (at 0.9125 0 180) (size 1.025 1.4) (layers "F.Cu" "F.Paste" "F.Mask") (roundrect_rratio 0.243902)
+      (net 21 "/A3N") (pintype "passive"))
+    (model "${KICAD6_3DMODEL_DIR}/Resistor_SMD.3dshapes/R_0805_2012Metric.wrl"
+      (offset (xyz 0 0 0))
+      (scale (xyz 1 1 1))
+      (rotate (xyz 0 0 0))
     )
   )
@@
   (segment (start 80.65 103.76) (end 80.65 108.1) (width 0.25) (layer "B.Cu") (net 19))
   (segment (start 80.65 108.1) (end 78.75 110) (width 0.25) (layer "B.Cu") (net 19))
+  (segment (start 73.8875 137.1) (end 73.8875 136.9875) (width 1) (layer "F.Cu") (net 21))
   (segment (start 74.5 123.75) (end 68.25 130) (width 0.2) (layer "F.Cu") (net 21))
+  (segment (start 68.25 131.35) (end 68.25 130) (width 1) (layer "F.Cu") (net 21))
   (segment (start 74.5 103) (end 74.5 123.75) (width 0.2) (layer "F.Cu") (net 21))
+  (segment (start 73.8875 136.9875) (end 68.25 131.35) (width 1) (layer "F.Cu") (net 21))
   (via (at 74.5 103) (size 0.8) (drill 0.4) (layers "F.Cu" "B.Cu") (net 21))
   (segment (start 73.5 102) (end 62.81 102) (width 0.2) (layer "B.Cu") (net 21))
@@
   (segment (start 74.5 103) (end 73.5 102) (width 0.2) (layer "B.Cu") (net 21))
   (segment (start 75.5 102.98995) (end 75 103.48995) (width 0.2) (layer "F.Cu") (net 22))
+  (segment (start 73.1 130) (end 70.75 130) (width 1) (layer "F.Cu") (net 22))
   (segment (start 75.5 102) (end 75.5 102.98995) (width 0.2) (layer "F.Cu") (net 22))
+  (segment (start 75.7125 137.1) (end 75.7125 132.6125) (width 1) (layer "F.Cu") (net 22))
   (segment (start 70.75 128.065686) (end 70.75 130) (width 0.2) (layer "F.Cu") (net 22))
   (segment (start 75 123.815686) (end 70.75 128.065686) (width 0.2) (layer "F.Cu") (net 22))
   (segment (start 75 103.48995) (end 75 123.815686) (width 0.2) (layer "F.Cu") (net 22))
+  (segment (start 75.7125 132.6125) (end 73.1 130) (width 1) (layer "F.Cu") (net 22))
   (via (at 75.5 102) (size 0.8) (drill 0.4) (layers "F.Cu" "B.Cu") (net 22))
   (segment (start 75 101.5) (end 64.85 101.5) (width 0.2) (layer "B.Cu") (net 22))
