File: hardware/Kicad/Controller V3/Pioneer Controller V3.kicad_pcb (KiCad board)
At the start: 2 copper layers, 72 x 98.8 mm, 27 parts, among them J1 Sensor Connector, J2 Power (IN), J4 Conn_Coaxial, SW1 SW_Push, SW2 SW_Push, SW5 SW_DIP_x02, U1 ESP32-S3, U2 2821, U3 DS3231_Precision_RTC, U4 RFM95W_LoRa_Radio_Transceiver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

Commit message: updated 5v
Connections:
- U1 pad 3V: +3V3 -> unconnected-(U1-Pad3V)
- U1 pad BAT: +5V -> unconnected-(U1-PadBAT)
- U1 pad USB: unconnected-(U1-PadUSB) -> +5V
- U2 pad 17: +5V -> unconnected-(U2-BAT-Pad17)
- U2 pad 19: unconnected-(U2-USB-Pad19) -> +5V
- U2 pad 2: +3V3 -> unconnected-(U2-3V-Pad2)
Routing:
- net +3V3: track 30.9 -> 0.00 mm, vias 2 -> 0
- net +5V: track 324.7 -> 334.6 mm
- net unconnected-(U1-Pad3V): track 0.00 -> 2.54 mm
Changed lines of the file:
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@@
   (net 1 "+5V")
   (net 2 "GND")
-  (net 3 "+3V3")
+  (net 3 "unconnected-(U1-Pad3V)")
   (net 4 "VIN")
   (net 5 "Net-(U7-SW)")
@@
   (net 27 "/SCL")
   (net 28 "/SDA")
-  (net 29 "unconnected-(U1-PadUSB)")
+  (net 29 "unconnected-(U1-PadBAT)")
   (net 30 "unconnected-(U2-ADC-Pad5)")
   (net 31 "unconnected-(U2-CHPD-Pad16)")
   (net 32 "unconnected-(U2-EN-Pad18)")
-  (net 33 "unconnected-(U2-USB-Pad19)")
+  (net 33 "unconnected-(U2-3V-Pad2)")
   (net 34 "unconnected-(U5-Pad3P3_V)")
   (net 35 "unconnected-(U3-Pad32K)")
@@
   (net 51 "unconnected-(U8-Pad3.3V)")
   (net 52 "unconnected-(U8-PadCD)")
+  (net 53 "unconnected-(U2-BAT-Pad17)")
   (footprint "Button_Switch_THT:SW_PUSH_6mm" (layer "F.Cu")
     (at 90.75 74.25 90)
@@
       (stroke (width 0.12) (type solid)) (fill none) (layer "Edge.Cuts"))
     (pad "3V" thru_hole circle (at 1.27 8.89 180) (size 1.524 1.524) (drill 0.762) (layers "*.Cu" "*.Mask")
-      (net 3 "+3V3") (pinfunction "3V") (pintype "input"))
+      (net 3 "unconnected-(U1-Pad3V)") (pinfunction "3V") (pintype "input+no_connect"))
     (pad "3V" thru_hole circle (at 1.27 11.43 180) (size 1.524 1.524) (drill 0.762) (layers "*.Cu" "*.Mask")
-      (net 3 "+3V3") (pinfunction "3V") (pintype "input"))
+      (net 3 "unconnected-(U1-Pad3V)") (pinfunction "3V") (pintype "input+no_connect"))
     (pad "A0" thru_hole circle (at 1.27 16.51 180) (size 1.524 1.524) (drill 0.762) (layers "*.Cu" "*.Mask")
       (net 14 "unconnected-(U1-PadA0)") (pinfunction "A0") (pintype "input+no_connect"))
@@
       (net 13 "/SW6") (pinfunction "A5") (pintype "input"))
     (pad "BAT" thru_hole circle (at 21.59 16.51 180) (size 1.524 1.524) (drill 0.762) (layers "*.Cu" "*.Mask")
-      (net 1 "+5V") (pinfunction "BAT") (pintype "input"))
+      (net 29 "unconnected-(U1-PadBAT)") (pinfunction "BAT") (pintype "input+no_connect"))
     (pad "D5" thru_hole circle (at 21.59 39.37 180) (size 1.524 1.524) (drill 0.762) (layers "*.Cu" "*.Mask")
       (net 49 "/CS1") (pinfunction "D5") (pintype "input"))
@@
       (net 9 "/TX") (pinfunction "TX") (pintype "input"))
     (pad "USB" thru_hole circle (at 21.59 21.59 180) (size 1.524 1.524) (drill 0.762) (layers "*.Cu" "*.Mask")
-      (net 29 "unconnected-(U1-PadUSB)") (pinfunction "USB") (pintype "input+no_connect"))
+      (net 1 "+5V") (pinfunction "USB") (pintype "input"))
   )
   (footprint "Capacitor_SMD:C_1206_3216Metric" (layer "F.Cu")
@@
       (net 18 "unconnected-(U2-RST-Pad1)") (pinfunction "RST") (pintype "input+no_connect"))
     (pad "2" thru_hole circle (at -16.51 10.16 90) (size 1.508 1.508) (drill 1) (layers "*.Cu" "*.Mask")
-      (net 3 "+3V3") (pinfunction "3V") (pintype "power_in"))
+      (net 33 "unconnected-(U2-3V-Pad2)") (pinfunction "3V") (pintype "power_in+no_connect"))
     (pad "3" thru_hole circle (at -13.97 10.16 90) (size 1.508 1.508) (drill 1) (layers "*.Cu" "*.Mask"))
     (pad "4" thru_hole circle (at -11.43 10.16 90) (size 1.508 1.508) (drill 1) (layers "*.Cu" "*.Mask")
@@
       (net 31 "unconnected-(U2-CHPD-Pad16)") (pinfunction "CHPD") (pintype "bidirectional+no_connect"))
     (pad "17" thru_hole circle (at -8.89 -10.16 90) (size 1.508 1.508) (drill 1) (layers "*.Cu" "*.Mask")
-      (net 1 "+5V") (pinfunction "BAT") (pintype "bidirectional"))
+      (net 53 "unconnected-(U2-BAT-Pad17)") (pinfunction "BAT") (pintype "bidirectional+no_connect"))
     (pad "18" thru_hole circle (at -6.35 -10.16 90) (size 1.508 1.508) (drill 1) (layers "*.Cu" "*.Mask")
       (net 32 "unconnected-(U2-EN-Pad18)") (pinfunction "EN") (pintype "input+no_connect"))
     (pad "19" thru_hole circle (at -3.81 -10.16 90) (size 1.508 1.508) (drill 1) (layers "*.Cu" "*.Mask")
-      (net 33 "unconnected-(U2-USB-Pad19)") (pinfunction "USB") (pintype "bidirectional+no_connect"))
+      (net 1 "+5V") (pinfunction "USB") (pintype "bidirectional"))
     (pad "20" thru_hole circle (at -1.27 -10.16 90) (size 1.508 1.508) (drill 1) (layers "*.Cu" "*.Mask")
       (net 47 "/SW2") (pinfunction "GPIO14") (pintype "bidirectional"))
@@
   (segment (start 84.08702 95.75) (end 82.8625 96.97452) (width 0.75) (layer "F.Cu") (net 1))
   (segment (start 92 97.425) (end 90.325 95.75) (width 0.75) (layer "F.Cu") (net 1))
+  (segment (start 35.56 78.12) (end 35.56 56.99) (width 0.75) (layer "F.Cu") (net 1))
   (segment (start 41.3075 93.5) (end 33.84 86.0325) (width 0.75) (layer "F.Cu") (net 1))
   (segment (start 90.75 50.75) (end 90.75 57.25) (width 0.4) (layer "F.Cu") (net 1))
-  (segment (start 31.745 58.255) (end 32.22 58.255) (width 0.75) (layer "F.Cu") (net 1))
   (segment (start 59 95.885) (end 59 103.75) (width 0.75) (layer "F.Cu") (net 1))
   (segment (start 55.88 78.105) (end 59.055 81.28) (width 0.75) (layer "F.Cu") (net 1))
   (segment (start 84.24 59.38) (end 86.36 61.5) (width 0.75) (layer "F.Cu") (net 1))
+  (segment (start 33.84 79.84) (end 35.56 78.12) (width 0.75) (layer "F.Cu") (net 1))
   (segment (start 75.565 95.885) (end 77.975 93.475) (width 0.75) (layer "F.Cu") (net 1))
   (segment (start 90.75 67.75) (end 90.75 74.25) (width 0.4) (layer "F.Cu") (net 1))
-  (segment (start 35.56 61.595) (end 35.56 78.12) (width 0.75) (layer "F.Cu") (net 1))
+  (segment (start 54.61 52.705) (end 58.735 52.705) (width 0.75) (layer "F.Cu") (net 1))
   (segment (start 89 66) (end 90.75 67.75) (width 0.4) (layer "F.Cu") (net 1))
   (segment (start 62.5325 92.3525) (end 63.235 92.3525) (width 0.75) (layer "F.Cu") (net 1))
-  (segment (start 54.715 57.89) (end 54.61 57.785) (width 0.75) (layer "F.Cu") (net 1))
   (segment (start 56.615 93.5) (end 41.3075 93.5) (width 0.75) (layer "F.Cu") (net 1))
   (segment (start 92 93.475) (end 87.25 93.475) (width 0.75) (layer "F.Cu") (net 1))
-  (segment (start 58.84 57.89) (end 54.715 57.89) (width 0.75) (layer "F.Cu") (net 1))
   (segment (start 59 95.885) (end 56.615 93.5) (width 0.75) (layer "F.Cu") (net 1))
   (segment (start 89 59) (end 89 66) (width 0.4) (layer "F.Cu") (net 1))
-  (segment (start 32.22 58.255) (end 35.56 61.595) (width 0.75) (layer "F.Cu") (net 1))
+  (segment (start 35.56 56.99) (end 31.745 53.175) (width 0.75) (layer "F.Cu") (net 1))
   (segment (start 63 107.75) (end 68.75 107.75) (width 0.75) (layer "F.Cu") (net 1))
-  (segment (start 35.56 78.12) (end 33.84 79.84) (width 0.75) (layer "F.Cu") (net 1))
+  (segment (start 58.735 52.705) (end 58.84 52.81) (width 0.75) (layer "F.Cu") (net 1))
   (segment (start 59 95.885) (end 75.565 95.885) (width 0.75) (layer "F.Cu") (net 1))
   (segment (start 70.82 109.82) (end 70.82 115) (width 0.75) (layer "F.Cu") (net 1))
@@
   (segment (start 59 95.885) (end 62.5325 92.3525) (width 0.75) (layer "F.Cu") (net 1))
   (segment (start 86.36 61.5) (end 86.36 67.31) (width 0.75) (layer "F.Cu") (net 1))
-  (via (at 54.61 57.785) (size 0.8) (drill 0.4) (layers "F.Cu" "B.Cu") (net 1))
+  (via (at 54.61 52.705) (size 0.8) (drill 0.4) (layers "F.Cu" "B.Cu") (net 1))
   (via (at 55.88 76.2) (size 0.8) (drill 0.4) (layers "F.Cu" "B.Cu") (net 1))
   (via (at 85.09 89.535) (size 0.8) (drill 0.4) (layers "F.Cu" "B.Cu") (net 1))
@@
   (segment (start 86.36 78.74) (end 86.995 79.375) (width 0.75) (layer "B.Cu") (net 1))
   (segment (start 81.915 58.11) (end 83.185 59.38) (width 0.75) (layer "B.Cu") (net 1))
-  (segment (start 54.61 57.785) (end 54.61 74.93) (width 0.75) (layer "B.Cu") (net 1))
-  (segment (start 54.61 74.93) (end 55.88 76.2) (width 0.75) (layer "B.Cu") (net 1))
+  (segment (start 54.61 52.705) (end 54.61 74.93) (width 0.75) (layer "B.Cu") (net 1))
   (segment (start 83.185 59.38) (end 84.24 59.38) (width 0.75) (layer "B.Cu") (net 1))
   (segment (start 59 86.87) (end 64.36 81.51) (width 0.75) (layer "B.Cu") (net 1))
   (segment (start 59 95.885) (end 59 86.87) (width 0.75) (layer "B.Cu") (net 1))
+  (segment (start 54.61 74.93) (end 55.88 76.2) (width 0.75) (layer "B.Cu") (net 1))
   (segment (start 84.699 32.11) (end 96.88 32.11) (width 0.75) (layer "B.Cu") (net 1))
   (segment (start 83.185 53.975) (end 81.915 55.245) (width 0.75) (layer "B.Cu") (net 1))
@@
   (segment (start 99.06 34.29) (end 99.06 44.45) (width 0.75) (layer "B.Cu") (net 1))
   (segment (start 86.36 67.31) (end 86.36 78.74) (width 0.75) (layer "B.Cu") (net 1))
-  (segment (start 52.065 63.335) (end 52.065 65.875) (width 0.75) (layer "F.Cu") (net 3))
-  (segment (start 52.535 65.405) (end 52.065 65.875) (width 0.75) (layer "F.Cu") (net 3))
-  (segment (start 58.42 65.405) (end 52.535 65.405) (width 0.75) (layer "F.Cu") (net 3))
-  (segment (start 79.16 65.51) (end 77.785 64.135) (width 0.75) (layer "F.Cu") (net 3))
-  (segment (start 77.785 64.135) (end 64.135 64.135) (width 0.75) (layer "F.Cu") (net 3))
-  (via (at 58.42 65.405) (size 0.8) (drill 0.4) (layers "F.Cu" "B.Cu") (net 3))
-  (via (at 64.135 64.135) (size 0.8) (drill 0.4) (layers "F.Cu" "B.Cu") (net 3))
-  (segment (start 59.69 64.135) (end 58.42 65.405) (width 0.75) (layer "B.Cu") (net 3))
-  (segment (start 64.135 64.135) (end 59.69 64.135) (width 0.75) (layer "B.Cu") (net 3))
+  (segment (start 52.065 63.335) (end 52.065 65.875) (width 0.25) (layer "F.Cu") (net 3))
   (segment (start 81.025 100.7875) (end 82.8625 98.95) (width 1) (layer "F.Cu") (net 4))
   (segment (start 80.95 111) (end 80.95 114.41) (width 1) (layer "F.Cu") (net 4))

Commit message: added some changes
Other:
- board text added: "5V"
- board text added: "Defender la alegría como una trinchera, un principio, una bandera, un destino, una certeza, un derecho. (M. Benedetti)"
- board text added: "F. Dallo & N. Zhao"
- board text added: "GND"
- board text added: "RX"
- board text added: "TX"
- board text removed: "4.7uF"

Commit message: more PCB updates
Parts:
- added G***: LOGO, LOGO, F.Cu at (41.9, 59.1)
Other:
- board text added: "VIN(5-32V)"

Commit message: feat: last kicad updates before sending order
Routing:
- net GND: track 0.00 -> 3.53 mm
Changed lines of the file:
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@@
   (segment (start 99.06 34.29) (end 99.06 44.45) (width 0.75) (layer "B.Cu") (net 1))
   (segment (start 86.36 67.31) (end 86.36 78.74) (width 0.75) (layer "B.Cu") (net 1))
+  (segment (start 85.1375 98.95) (end 83.975 100.1125) (width 0.25) (layer "F.Cu") (net 2))
+  (segment (start 83.975 100.1125) (end 83.975 102) (width 0.25) (layer "F.Cu") (net 2))
   (segment (start 52.065 63.335) (end 52.065 65.875) (width 0.25) (layer "F.Cu") (net 3))
   (segment (start 81.025 100.7875) (end 82.8625 98.95) (width 1) (layer "F.Cu") (net 4))
